Commit message: Removed texture -- not working

File: rosplane_sim/agents/myTwinDream/myTwinDream.xacro (robot description, xacro)
@@ -36,11 +36,4 @@
         </xacro:unless>
       </geometry>
-      <material name="wing_material">
-        <script>
-          <uri>package://rosplane_sim/agents/$(arg mav_name)/materials/scripts</uri>
-          <uri>package://rosplane_sim/agents/$(arg mav_name)/materials/textures</uri>
-          <name>wing/texture</name>
-        </script>
-      </material>
     </visual>
     <collision name="plane_collision">

Commit message: Added truth plugin

File: rosplane_sim/agents/myTwinDream/myTwinDream.xacro (robot description, xacro)
@@ -44,5 +44,5 @@
     </collision>
     <!-- Wheels -->
-    <!-- <xacro:include filename="$(find fcu_sim_plugins)/xacro/wheel.xacro"/>
+    <xacro:include filename="$(find fcu_sim_plugins)/xacro/wheel.xacro"/>
     <xacro:caster
       radius="0.05">
@@ -56,6 +56,12 @@
       radius="0.02">
       <origin xyz="-${body_length*0.54} 0 -${body_height*0.15}"/>
-    </xacro:caster> -->
+    </xacro:caster>
   </link>
+  <!-- Simulator Truth -->
+  <xacro:include filename="$(find rosplane_sim)/xacro/aircraft_truth.xacro"/>
+  <xacro:aircraft_truth
+    namespace="${namespace}"
+    parent_link="${namespace}/base_link"
+    wind_speed_topic="gazebo/wind_speed"/>
   <!-- Aerodynamics -->
   <xacro:include filename="$(find fcu_sim_plugins)/xacro/aircraft_forces_and_moments.xacro"/>
@@ -64,4 +70,34 @@
     parent_link="${namespace}/base_link"
     command_topic="command"/>
+  <!-- GPS -->
+  <!-- <xacro:include filename="$(find fcu_sim_plugins)/xacro/GPS.xacro"/>
+  <xacro:GPS_BYU
+    namespace="${namespace}"
+    parent_link="${namespace}/base_link"
+    GPS_topic="gps/data"
+    update_rate="1">
+  </xacro:GPS_BYU> -->
+  <!-- IMU -->
+  <!-- <xacro:include filename="$(find fcu_sim_plugins)/xacro/imu.xacro"/>
+  <xacro:IMU_MPU6050
+    namespace="${namespace}"
+    parent_link="${namespace}/base_link"
+    imu_topic="imu/data"
+    update_rate="500">
+  </xacro:IMU_MPU6050> -->
+  <!-- Airspeed -->
+  <!-- <xacro:include filename="$(find fcu_sim_plugins)/xacro/airspeed.xacro"/>
+  <xacro:airspeed_MPXV5004G
+    namespace="${namespace}"
+    parent_link="${namespace}/base_link"
+    airspeed_topic="airspeed/data">
+  </xacro:airspeed_MPXV5004G> -->
+  <!-- Barometer -->
+  <!-- <xacro:include filename="$(find fcu_sim_plugins)/xacro/barometer.xacro"/>
+  <xacro:Barometer_MS5611
+    namespace="${namespace}"
+    parent_link="${namespace}/base_link"
+    baro_topic="baro/data">
+  </xacro:Barometer_MS5611> -->
   <!-- Chase Camera -->
   <xacro:include filename="$(find fcu_sim_plugins)/xacro/camera.xacro"/>
@@ -75,16 +111,6 @@
     <origin xyz="-${1.1*body_length} 0 ${0.8*body_height}"/>
   </xacro:simple_camera>
-  <!-- Color -->
-  <gazebo reference="${namespace}/base_link">
-    <material>Gazebo/Blue</material>
-  </gazebo>
-  <!-- Sensors -->
-  <xacro:include filename="$(find fcu_sim_plugins)/xacro/aircraft_truth.xacro"/>
-  <xacro:aircraft_truth
-    namespace="${namespace}"
-    parent_link="${namespace}/base_link"
-    wind_speed_topic="gazebo/wind_speed"/>
   <!-- Gimbal -->
-  <xacro:include filename="$(find fcu_sim_plugins)/xacro/gimbal.xacro"/>
+  <!-- <xacro:include filename="$(find fcu_sim_plugins)/xacro/gimbal.xacro"/>
   <xacro:gimbal_ZENMUSE
     namespace="${namespace}"
@@ -96,29 +122,7 @@
     use_slipring="true">
     <origin xyz="-${0.4*body_length} 0 -${0.4*body_height}" rpy="0 0 0"/>
-  </xacro:gimbal_ZENMUSE>
-  <!-- Airspeed -->
-  <xacro:include filename="$(find fcu_sim_plugins)/xacro/airspeed.xacro"/>
-  <xacro:airspeed_MPXV5004G
-    namespace="${namespace}"
-    parent_link="${namespace}/base_link"
-    airspeed_topic="airspeed/data">
-  </xacro:airspeed_MPXV5004G>
-  <!-- GPS -->
-  <xacro:include filename="$(find fcu_sim_plugins)/xacro/GPS.xacro"/>
-  <xacro:GPS_BYU
-    namespace="${namespace}"
-    parent_link="${namespace}/base_link"
-    GPS_topic="gps/data"
-    update_rate="1">
-  </xacro:GPS_BYU>
-  <!-- Barometer -->
-  <xacro:include filename="$(find fcu_sim_plugins)/xacro/barometer.xacro"/>
-  <xacro:Barometer_MS5611
-    namespace="${namespace}"
-    parent_link="${namespace}/base_link"
-    baro_topic="baro/data">
-  </xacro:Barometer_MS5611>
+  </xacro:gimbal_ZENMUSE> -->
   <!-- Sonar -->
-  <xacro:include filename="$(find fcu_sim_plugins)/xacro/sonar.xacro"/>
+  <!-- <xacro:include filename="$(find fcu_sim_plugins)/xacro/sonar.xacro"/>
   <xacro:Sonar_MB1030
     namespace="${namespace}"
@@ -126,12 +130,4 @@
     sonar_topic="sonar/data">
     <origin xyz="0 0 0" rpy="0 0 0"/>
-  </xacro:Sonar_MB1030>
-  <!-- IMU -->
-  <xacro:include filename="$(find fcu_sim_plugins)/xacro/imu.xacro"/>
-  <xacro:IMU_MPU6050
-    namespace="${namespace}"
-    parent_link="${namespace}/base_link"
-    imu_topic="imu/data"
-    update_rate="500">
-  </xacro:IMU_MPU6050>
+  </xacro:Sonar_MB1030> -->
 </robot>
