Commit message: Restructured package to match roscopter and rosflight

File: rosplane_sim/xacro/default_fixedwing.xacro (robot description, xacro)
@@ -6,5 +6,5 @@
   <xacro:property name="command_topic" value="command"/>
   <xacro:property name="use_mesh_file" value="true" />
-  <xacro:property name="mesh_file" value="package://rosplane_sim/agents/$(arg mav_name)/meshes/default_fixedwing.dae"/>
+  <xacro:property name="mesh_file" value="package://rosplane_sim/xacro/default_fixedwing.dae"/>
   <xacro:property name="body_width" value="1.4"/>
   <xacro:property name="body_height" value="1.0" />
@@ -44,5 +44,5 @@
     </collision>
     <!-- Wheels -->
-    <xacro:include filename="$(find rosplane_sim)/xacro/wheel.xacro"/>
+    <!-- <xacro:include filename="$(find rosplane_sim)/xacro/wheel.xacro"/>
     <xacro:caster
       radius="0.05">
@@ -56,5 +56,5 @@
       radius="0.02">
       <origin xyz="-${body_length*0.54} 0 -${body_height*0.15}"/>
-    </xacro:caster>
+    </xacro:caster> -->
   </link>
   <!-- Simulator Truth -->
@@ -101,5 +101,5 @@
   </xacro:Barometer_MS5611> -->
   <!-- Chase Camera -->
-  <xacro:include filename="$(find fcu_sim_plugins)/xacro/camera.xacro"/>
+  <!-- <xacro:include filename="$(find fcu_sim_plugins)/xacro/camera.xacro"/>
   <xacro:simple_camera
     namespace="${namespace}/chase"
@@ -110,5 +110,5 @@
     image_camera_info_topic="camera_info">
     <origin xyz="-${1.1*body_length} 0 ${0.8*body_height}"/>
-  </xacro:simple_camera>
+  </xacro:simple_camera> -->
   <!-- Gimbal -->
   <!-- <xacro:include filename="$(find fcu_sim_plugins)/xacro/gimbal.xacro"/>
