Commit message: Moved aircraft xacro using design model to xacro folder

File: rosplane_sim/xacro/design_model.xacro (robot description, xacro)
@@ -5,5 +5,5 @@
       name="Design_Model"
       params="namespace parent_link command_topic">
-      <xacro:aircraft_forces_and_moments_macro
+      <xacro:design_model_macro
         namespace="${namespace}"
         parent_link="${namespace}/base_link"
@@ -11,13 +11,13 @@
         command_topic="${command_topic}"
         parent_frame_id="${namespace}/base_link">
-      </xacro:aircraft_forces_and_moments_macro>
+      </xacro:design_model_macro>
     </xacro:macro>
   <!-- Macro to add the simplified dynamics from the design model. -->
-  <xacro:macro name="aircraft_forces_and_moments_macro"
+  <xacro:macro name="design_model_macro"
     params="namespace  parent_link wind_speed_topic command_topic parent_frame_id">
     <gazebo>
       <plugin
-        filename="libaircraft_forces_and_moments_plugin.so"
-        name="${namespace}_aircraft_forces_and_moments">
+        filename="libdesign_model_plugin.so"
+        name="${namespace}_design_model">
         <linkName>${parent_link}</linkName>
         <namespace>${namespace}</namespace>
