Commit message: Migrate plugins to rosflight_plugins and rosparam server (#35)
* Migrated all plugins to rosflight_plugins package 

Also moved all parameters to yaml file, rather than using sdf param server.

* Updated yaml

* Added plugin default params

* Migrated all plugins to rosflight_plugins package 

Also moved all parameters to yaml file, rather than using sdf param server.

* Updated yaml

* Added plugin default params

File: rosplane_sim/xacro/aircraft_forces_and_moments.xacro (robot description, xacro)
@@ -3,17 +3,14 @@
     <!-- Forces And Moments Plugin -->
     <xacro:macro
-      name="myTwinDream"
-      params="namespace parent_link command_topic">
+      name="aircraft_dynamics"
+      params="namespace parent_link">
       <xacro:aircraft_forces_and_moments_macro
         namespace="${namespace}"
-        parent_link="${namespace}/base_link"
-        wind_speed_topic="gazebo/wind_speed"
-        command_topic="${command_topic}"
-        parent_frame_id="${namespace}/base_link">
+        parent_link="${namespace}/base_link">
       </xacro:aircraft_forces_and_moments_macro>
     </xacro:macro>
   <!-- Macro to add a generic odometry sensor. -->
   <xacro:macro name="aircraft_forces_and_moments_macro"
-    params="namespace  parent_link wind_speed_topic command_topic parent_frame_id">
+    params="namespace parent_link">
     <gazebo>
       <plugin
@@ -22,7 +19,4 @@
         <linkName>${parent_link}</linkName>
         <namespace>${namespace}</namespace>
-        <windSpeedTopic>${wind_speed_topic}</windSpeedTopic>
-        <commandTopic>${command_topic}</commandTopic>
-        <parentFrameId>${parent_frame_id}</parentFrameId>
       </plugin>
     </gazebo>

File: rosplane_sim/xacro/aircraft_truth.xacro (robot description, xacro)
@@ -4,10 +4,9 @@
     <xacro:macro
       name="aircraft_truth"
-      params="namespace parent_link wind_speed_topic">
+      params="namespace parent_link">
       <gazebo>
         <plugin filename="libaircraft_truth_plugin.so" name="${namespace}_aircraft_truth_plugin">
           <namespace>${namespace}</namespace>
           <linkName>${namespace}/base_link</linkName>
-          <windSpeedTopic>${wind_speed_topic}</windSpeedTopic>
         </plugin>
       </gazebo>

File: rosplane_sim/xacro/default_fixedwing.xacro (robot description, xacro)
@@ -62,42 +62,34 @@
   <xacro:aircraft_truth
     namespace="${namespace}"
-    parent_link="${namespace}/base_link"
-    wind_speed_topic="gazebo/wind_speed"/>
+    parent_link="${namespace}/base_link"/>
   <!-- Aerodynamics -->
   <xacro:include filename="$(find rosplane_sim)/xacro/aircraft_forces_and_moments.xacro"/>
-  <xacro:myTwinDream
+  <xacro:aircraft_dynamics
     namespace="${namespace}"
-    parent_link="${namespace}/base_link"
-    command_topic="command"/>
+    parent_link="${namespace}/base_link"/>
   <!-- GPS -->
-  <!-- <xacro:include filename="$(find fcu_sim_plugins)/xacro/GPS.xacro"/>
-  <xacro:GPS_BYU
+  <xacro:include filename="$(find rosflight_plugins)/xacro/GPS.xacro"/>
+  <xacro:gps_plugin_macro
     namespace="${namespace}"
-    parent_link="${namespace}/base_link"
-    GPS_topic="gps/data"
-    update_rate="1">
-  </xacro:GPS_BYU> -->
+    parent_link="${namespace}/base_link">
+  </xacro:gps_plugin_macro>
   <!-- IMU -->
-  <!-- <xacro:include filename="$(find fcu_sim_plugins)/xacro/imu.xacro"/>
-  <xacro:IMU_MPU6050
+  <xacro:include filename="$(find rosflight_plugins)/xacro/imu.xacro"/>
+  <xacro:imu_plugin_macro
     namespace="${namespace}"
-    parent_link="${namespace}/base_link"
-    imu_topic="imu/data"
-    update_rate="500">
-  </xacro:IMU_MPU6050> -->
+    parent_link="${namespace}/base_link">
+  </xacro:imu_plugin_macro>
   <!-- Airspeed -->
-  <!-- <xacro:include filename="$(find fcu_sim_plugins)/xacro/airspeed.xacro"/>
-  <xacro:airspeed_MPXV5004G
+  <xacro:include filename="$(find rosflight_plugins)/xacro/airspeed.xacro"/>
+  <xacro:airspeed_plugin_macro
     namespace="${namespace}"
-    parent_link="${namespace}/base_link"
-    airspeed_topic="airspeed/data">
-  </xacro:airspeed_MPXV5004G> -->
+    parent_link="${namespace}/base_link">
+  </xacro:airspeed_plugin_macro>
   <!-- Barometer -->
-  <!-- <xacro:include filename="$(find fcu_sim_plugins)/xacro/barometer.xacro"/>
-  <xacro:Barometer_MS5611
+  <xacro:include filename="$(find rosflight_plugins)/xacro/barometer.xacro"/>
+  <xacro:barometer_plugin_macro
     namespace="${namespace}"
-    parent_link="${namespace}/base_link"
-    baro_topic="baro/data">
-  </xacro:Barometer_MS5611> -->
+    parent_link="${namespace}/base_link">
+  </xacro:barometer_plugin_macro>
   <!-- Chase Camera -->
   <!-- <xacro:include filename="$(find fcu_sim_plugins)/xacro/camera.xacro"/>
@@ -123,11 +115,3 @@
     <origin xyz="-${0.4*body_length} 0 -${0.4*body_height}" rpy="0 0 0"/>
   </xacro:gimbal_ZENMUSE> -->
-  <!-- Sonar -->
-  <!-- <xacro:include filename="$(find fcu_sim_plugins)/xacro/sonar.xacro"/>
-  <xacro:Sonar_MB1030
-    namespace="${namespace}"
-    parent_link="${namespace}/base_link"
-    sonar_topic="sonar/data">
-    <origin xyz="0 0 0" rpy="0 0 0"/>
-  </xacro:Sonar_MB1030> -->
 </robot>
